File: pcb/kicad.kicad_pcb (KiCad board)
At the start: 2 copper layers, 42.9 x 62.9 mm, 7 parts, among them SW1 SW_Push, SW2 SW_Push, SW3 SW_Push, SW4 SW_Push, U1 XIAO-RP2040-DIP

Commit message: update cad and pcb to include lcd display
Parts:
- added OLED_0.1: ~, OLED_0.91inch:SSD1306-0.91-OLED-4pin-128x32, F.Cu at (157.3, 92.7)
Connections:
- U1 pad 12: unconnected-(U1-3V3-Pad12) -> Net-(OLED_0.1-VCC_IN)
- U1 pad 6: unconnected-(U1-GPIO7/SCL-Pad6) -> Net-(OLED_0.1-SCL)
Routing:
- net Net-(D1-DIN): track 5.60 -> 56.2 mm
- net Net-(OLED_0.1-SCL): track 0.00 -> 47.4 mm
- net Net-(OLED_0.1-VCC_IN): track 0.00 -> 25.2 mm
- net GND: track 80.5 -> 93.3 mm
Other:
- board size 42.9 x 62.9 mm -> 59.5 x 62.9 mm
